File: picoface_16v8.kicad_pcb (KiCad board)
At the start: 2 copper layers, 79.2 x 69.6 mm, 23 parts, among them J1 ZX_Spectrum_Connector_48K_SOR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, J2 DE9_Plug, Q1 DMG2305, SW1 SW_USER, SW2 SW_RESET, SW3 SW_RUN, U2 Pico, U3 74LS240

Commit message: Correct resistor typo and add GALASM to schematic
I just blindly typed in 8K1 whereas the resistor I have are 8K2.
Parts:
- R1, R2, R3, R4, R5, R7, R8: value 8K1 -> 8K2
Changed lines of the file:
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@@
 			)
 		)
-		(property "Value" "8K1"
+		(property "Value" "8K2"
 			(at 3.81 1.92 90)
 			(layer "F.Fab")
@@
 			)
 		)
-		(property "Value" "8K1"
+		(property "Value" "8K2"
 			(at 3.81 1.92 90)
 			(layer "F.Fab")
@@
 			)
 		)
-		(property "Value" "8K1"
+		(property "Value" "8K2"
 			(at 3.81 1.92 90)
 			(layer "F.Fab")
@@
 			)
 		)
-		(property "Value" "8K1"
+		(property "Value" "8K2"
 			(at 3.81 1.92 90)
 			(layer "F.Fab")
@@
 			)
 		)
-		(property "Value" "8K1"
+		(property "Value" "8K2"
 			(at 3.81 1.92 90)
 			(layer "F.Fab")
@@
 			)
 		)
-		(property "Value" "8K1"
+		(property "Value" "8K2"
 			(at 3.81 1.92 90)
 			(layer "F.Fab")
@@
 			)
 		)
-		(property "Value" "8K1"
+		(property "Value" "8K2"
 			(at 3.81 1.92 90)
 			(layer "F.Fab")
