File: picoface_16v8.kicad_sch (KiCad schematic)
At the start: 23 parts, among them J1 ZX_Spectrum_Connector_48K_SOR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, J2 DE9_Plug, Q1 DMG2305, SW1 SW_USER, SW2 SW_RESET, SW3 SW_RUN, U2 Pico, U3 74LS240

Commit message: Update to KiCad 9 and add missing gerbers
See issue #1 for details
Parts:
- J1: footprint 8bits:ZX_CONN -> mysyms:ZX_CONN
- J2: footprint 8bits:DSUB-9_Female_Vertical_P2.77x2.84mm_MountingHoles -> mysyms:DSUB-9_Female_Vertical_P2.77x2.84mm_MountingHoles
